File: lib/controll.sch (EAGLE design)
At the start: 2 parts, among them U1 AL5802-7, U4 AL5802-7

Commit message: adds H-bridge
Parts:
- added U$1: CHIP_PRO, CHIP_Pro-Footprint:CHIP_PRO
Connections:
- net VCC renamed 24V
- new net N$4: U4.GND
- new net N$7: U4.EN
- new net N$8: U4.OUT
- net GND: now also U$1.AGND, U$1.GND@0, U$1.GND@2, U$1.GND@3, U$1.GND@4, U$1.GND@5, U$1.GND@6, U$1.GND@7; no longer U4.GND
- net N$1: no longer U4.OUT
- net N$5: no longer U4.EN
