File: control1.brd (EAGLE design)
At the start: 195 x 35 mm, 63 parts

Commit message: Revert "Merge remote-tracking branch 'refs/remotes/origin/master' into new-layout"
This reverts commit d786cf153478cbc5e1d0f0cbdb23b775e7a3effd.
Parts:
- U$39: value MOTORCONNECTOR -> SFV18R-3STBE1HLF; device Smile_Shade:MOTORCONNECTOR -> Smile_Shade:SFV18R-3STBE1HLF
- moved U$38 109.2 mm to (80.5, 48.5), turned to 90 degrees
- moved U$39 48.9 mm to (174.0, -15.0), turned to 180 degrees
- moved C2 13.9 mm to (92.0, 24.0)
- moved U$2 11.4 mm to (79.3, 31.0)
- moved U$35 9.90 mm to (103.5, 25.0)
- moved C1 4.47 mm to (51.5, 21.0), flipped to the bottom
- moved U$1 3.00 mm to (25.4, 15.8)
Connections:
- net LEDSTR_1: now also U$39.P$18
- net LEDSTR_10: now also U$39.P$9
- net LEDSTR_11: now also U$39.P$10
- net LEDSTR_12: now also U$39.P$7
- net LEDSTR_13: now also U$39.P$6
- net LEDSTR_14: now also U$39.P$5
- net LEDSTR_15: now also U$39.P$4
- net LEDSTR_16: now also U$39.P$3
- net LEDSTR_17: now also U$39.P$1
- net LEDSTR_18: now also U$39.P$2
- net LEDSTR_2: now also U$39.P$17
- net LEDSTR_3: now also U$39.P$16
- net LEDSTR_4: now also U$39.P$15
- net LEDSTR_5: now also U$39.P$12
- net LEDSTR_6: now also U$39.P$13
- net LEDSTR_7: now also U$39.P$14
- net LEDSTR_8: now also U$39.P$11
- net LEDSTR_9: now also U$39.P$8
- net M1A: no longer U$38.P$2
- net M1B: no longer U$38.P$1
- net M2A: now also U$38.P$1; no longer U$39.P$1
- net M2B: now also U$38.P$2; no longer U$39.P$2
Routing:
- net GND: track 135.7 -> 2.15 mm, vias 1 -> 0
- net 48V: track 194.0 -> 61.8 mm
- net ZN8: track 77.5 -> 0.00 mm, vias 1 -> 0
- net ZN0: track 60.7 -> 0.00 mm, vias 1 -> 0
- net ZN1: track 56.9 -> 0.00 mm, vias 1 -> 0
- net ZN9: track 51.7 -> 0.00 mm, vias 1 -> 0
- net ZN2: track 47.3 -> 0.00 mm, vias 1 -> 0
- net ZN10: track 43.8 -> 0.00 mm, vias 1 -> 0
- net ZN3: track 41.6 -> 0.00 mm, vias 1 -> 0
- net ZN11: track 35.9 -> 0.00 mm, vias 1 -> 0
- net ZN4: track 32.0 -> 0.00 mm, vias 1 -> 0
- net ZN12: track 28.0 -> 0.00 mm, vias 1 -> 0
- net ZN5: track 24.3 -> 0.00 mm, vias 1 -> 0
- net ZN13: track 20.1 -> 0.00 mm, vias 1 -> 0
- net ZN6: track 16.7 -> 0.00 mm, vias 1 -> 0
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Other:
- board size 195 x 35 mm -> 188 x 32 mm
