File: strip14.brd (EAGLE design)
At the start: 288.4 x 6 mm, 10 parts

Commit message: setts up warm cool LED support
Parts:
- added U$11, U$12, U$13, U$14, U$15, U$16, U$17, U$18, U$19, U$20: BXEN-40E-11M-3A-00-0-0, Smile_Shade:BXEN-40E-11M-3A-00-0-0
Connections:
- new net N$10: U$19.P$2, U$20.P$1
- new net N$11: U$18.P$2, U$19.P$1
- new net N$12: U$17.P$2, U$18.P$1
- new net N$13: U$16.P$2, U$17.P$1
- new net N$14: U$15.P$2, U$16.P$1
- new net N$15: U$11.P$2, U$12.P$1
- new net N$16: U$12.P$2, U$13.P$1
- new net N$17: U$13.P$2, U$14.P$1
- new net N$18: U$14.P$2, U$15.P$1
Other:
- board size 288.4 x 6 mm -> 290 x 11 mm
Changed lines of the file:
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@@
 <?xml version="1.0" encoding="utf-8"?>
 <!DOCTYPE eagle SYSTEM "eagle.dtd">
-<eagle version="8.0.0">
+<eagle version="8.0.2">
 <drawing>
 <settings>
@@
 <setting verticaltext="up"/>
 </settings>
-<grid distance="1" unitdist="mm" unit="mm" style="lines" multiple="1" display="yes" altdistance="1.2" altunitdist="inch" altunit="inch"/>
+<grid distance="1" unitdist="mm" unit="mm" style="lines" multiple="1" display="yes" altdistance="1" altunitdist="mm" altunit="mm"/>
 <layers>
 <layer number="1" name="Top" color="4" fill="1" visible="yes" active="yes"/>
@@
 <board>
 <plain>
-<wire x1="0" y1="0" x2="288.41" y2="0" width="0" layer="20"/>
-<wire x1="288.41" y1="0" x2="288.41" y2="6.02" width="0" layer="20"/>
-<wire x1="288.41" y1="6.02" x2="0" y2="6.02" width="0" layer="20"/>
-<wire x1="0" y1="6.02" x2="0" y2="0" width="0" layer="20"/>
-<dimension x1="0" y1="0" x2="0" y2="6.02" x3="-2" y3="3.01" textsize="1.778" layer="1"/>
-<dimension x1="0" y1="6.02" x2="289" y2="6" x3="144.50006875" y3="7.01" textsize="1.778" layer="1"/>
+<wire x1="0" y1="0" x2="290" y2="0" width="0" layer="20"/>
+<wire x1="290" y1="0" x2="290" y2="11.02" width="0" layer="20"/>
+<wire x1="290" y1="11.02" x2="0" y2="11.02" width="0" layer="20"/>
+<wire x1="0" y1="11.02" x2="0" y2="0" width="0" layer="20"/>
+<dimension x1="0" y1="0" x2="0" y2="11.02" x3="-2" y3="5.51" textsize="1.778" layer="1"/>
+<dimension x1="0" y1="11.02" x2="290" y2="11" x3="145.00006875" y3="12.010003125" textsize="1.778" layer="1"/>
 </plain>
 <attributes>
@@
 <element name="U$9" library="Smile_Shade" package="JDSTS2.EM-HRHT-XX52-1" value="JDSTS2.EM-HRHT-XX52-1" x="249.84" y="3"/>
 <element name="U$10" library="Smile_Shade" package="JDSTS2.EM-HRHT-XX52-1" value="JDSTS2.EM-HRHT-XX52-1" x="280.32" y="3"/>
+<element name="U$11" library="Smile_Shade" package="BXEN-40E-11M-3A-00-0-0" value="BXEN-40E-11M-3A-00-0-0" x="6.2" y="5.3"/>
+<element name="U$12" library="Smile_Shade" package="BXEN-40E-11M-3A-00-0-0" value="BXEN-40E-11M-3A-00-0-0" x="0" y="-11"/>
+<element name="U$13" library="Smile_Shade" package="BXEN-40E-11M-3A-00-0-0" value="BXEN-40E-11M-3A-00-0-0" x="0" y="-18"/>
+<element name="U$14" library="Smile_Shade" package="BXEN-40E-11M-3A-00-0-0" value="BXEN-40E-11M-3A-00-0-0" x="0" y="-25"/>
+<element name="U$15" library="Smile_Shade" package="BXEN-40E-11M-3A-00-0-0" value="BXEN-40E-11M-3A-00-0-0" x="0" y="-32"/>
+<element name="U$16" library="Smile_Shade" package="BXEN-40E-11M-3A-00-0-0" value="BXEN-40E-11M-3A-00-0-0" x="0" y="-39"/>
+<element name="U$17" library="Smile_Shade" package="BXEN-40E-11M-3A-00-0-0" value="BXEN-40E-11M-3A-00-0-0" x="0" y="-46"/>
+<element name="U$18" library="Smile_Shade" package="BXEN-40E-11M-3A-00-0-0" value="BXEN-40E-11M-3A-00-0-0" x="0" y="-53"/>
+<element name="U$19" library="Smile_Shade" package="BXEN-40E-11M-3A-00-0-0" value="BXEN-40E-11M-3A-00-0-0" x="0" y="-60"/>
+<element name="U$20" library="Smile_Shade" package="BXEN-40E-11M-3A-00-0-0" value="BXEN-40E-11M-3A-00-0-0" x="0" y="-67"/>
 </elements>
 <signals>
@@
 <wire x1="249.84" y1="3" x2="283.32" y2="3" width="0" layer="19" extent="1-1"/>
 </signal>
+<signal name="N$10">
+<contactref element="U$20" pad="P$1"/>
+<contactref element="U$19" pad="P$2"/>
+<wire x1="1.55" y1="-60" x2="-1.1" y2="-67" width="0" layer="19" extent="1-1"/>
+</signal>
+<signal name="N$11">
+<contactref element="U$19" pad="P$1"/>
+<contactref element="U$18" pad="P$2"/>
+<wire x1="1.55" y1="-53" x2="-1.1" y2="-60" width="0" layer="19" extent="1-1"/>
+</signal>
+<signal name="N$12">
+<contactref element="U$18" pad="P$1"/>
+<contactref element="U$17" pad="P$2"/>
+<wire x1="1.55" y1="-46" x2="-1.1" y2="-53" width="0" layer="19" extent="1-1"/>
+</signal>
+<signal name="N$13">
+<contactref element="U$17" pad="P$1"/>
+<contactref element="U$16" pad="P$2"/>
+<wire x1="1.55" y1="-39" x2="-1.1" y2="-46" width="0" layer="19" extent="1-1"/>
+</signal>
+<signal name="N$14">
+<contactref element="U$16" pad="P$1"/>
+<contactref element="U$15" pad="P$2"/>
+<wire x1="1.55" y1="-32" x2="-1.1" y2="-39" width="0" layer="19" extent="1-1"/>
+</signal>
+<signal name="N$15">
+<contactref element="U$11" pad="P$2"/>
+<contactref element="U$12" pad="P$1"/>
+<wire x1="7.75" y1="5.3" x2="-1.1" y2="-11" width="0" layer="19" extent="1-1"/>
+</signal>
+<signal name="N$16">
+<contactref element="U$12" pad="P$2"/>
+<contactref element="U$13" pad="P$1"/>
+<wire x1="1.55" y1="-11" x2="-1.1" y2="-18" width="0" layer="19" extent="1-1"/>
+</signal>
+<signal name="N$17">
+<contactref element="U$13" pad="P$2"/>
+<contactref element="U$14" pad="P$1"/>
+<wire x1="1.55" y1="-18" x2="-1.1" y2="-25" width="0" layer="19" extent="1-1"/>
+</signal>
+<signal name="N$18">
+<contactref element="U$14" pad="P$2"/>
+<contactref element="U$15" pad="P$1"/>
+<wire x1="1.55" y1="-25" x2="-1.1" y2="-32" width="0" layer="19" extent="1-1"/>
+</signal>
 </signals>
